File: PolicyBadge/PolicyBadge25/boost.kicad_sch (KiCad schematic)
At the start: 9 parts, among them U3 TPS613222ADBVR

Commit message: Released version of PCB
Parts:
- U4: renamed from U3; FT Rotation Offset (none) -> 180
- renumbered C7 to C3, C6 to C4, C1 to C5, C2 to C6, C5 to C7, R5 to R13
Changed lines of the file:
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@@
 		(dnp no)
 		(fields_autoplaced yes)
-		(property "Reference" "C2"
+		(property "Reference" "C6"
 			(at 186.69 116.8399 90)
 			(effects
@@
 			(project "PolicyBadge25"
 				(path "/3911717a-8f19-42c2-8f04-ebfae4e12db6/7d9e9d91-9070-4e08-95e2-83714d549a8d"
-					(reference "C2")
+					(reference "C6")
 					(unit 1)
 				)
@@
 		(dnp no)
 		(fields_autoplaced yes)
-		(property "Reference" "#PWR026"
+		(property "Reference" "#PWR033"
 			(at 93.98 133.35 0)
 			(effects
@@
 			(project "PolicyBadge25"
 				(path "/3911717a-8f19-42c2-8f04-ebfae4e12db6/7d9e9d91-9070-4e08-95e2-83714d549a8d"
-					(reference "#PWR026")
+					(reference "#PWR033")
 					(unit 1)
 				)
@@
 		(dnp no)
 		(fields_autoplaced yes)
-		(property "Reference" "#PWR023"
+		(property "Reference" "#PWR036"
 			(at 182.88 133.35 0)
 			(effects
@@
 			(project ""
 				(path "/3911717a-8f19-42c2-8f04-ebfae4e12db6/7d9e9d91-9070-4e08-95e2-83714d549a8d"
-					(reference "#PWR023")
+					(reference "#PWR036")
 					(unit 1)
 				)
@@
 		(dnp no)
 		(fields_autoplaced yes)
-		(property "Reference" "#PWR024"
+		(property "Reference" "#PWR035"
 			(at 128.27 133.35 0)
 			(effects
@@
 			(project "PolicyBadge25"
 				(path "/3911717a-8f19-42c2-8f04-ebfae4e12db6/7d9e9d91-9070-4e08-95e2-83714d549a8d"
-					(reference "#PWR024")
+					(reference "#PWR035")
 					(unit 1)
 				)
@@
 		(dnp no)
 		(fields_autoplaced yes)
-		(property "Reference" "C1"
+		(property "Reference" "C5"
 			(at 172.72 116.8399 90)
 			(effects
@@
 			(project ""
 				(path "/3911717a-8f19-42c2-8f04-ebfae4e12db6/7d9e9d91-9070-4e08-95e2-83714d549a8d"
-					(reference "C1")
+					(reference "C5")
 					(unit 1)
 				)
@@
 		(dnp no)
 		(fields_autoplaced yes)
-		(property "Reference" "C7"
+		(property "Reference" "C3"
 			(at 107.95 114.2999 90)
 			(effects
@@
 			(project ""
 				(path "/3911717a-8f19-42c2-8f04-ebfae4e12db6/7d9e9d91-9070-4e08-95e2-83714d549a8d"
-					(reference "C7")
+					(reference "C3")
 					(unit 1)
 				)
@@
 		(dnp no)
 		(fields_autoplaced yes)
-		(property "Reference" "R5"
+		(property "Reference" "R13"
 			(at 143.51 73.66 0)
 			(effects
@@
 			(project ""
 				(path "/3911717a-8f19-42c2-8f04-ebfae4e12db6/7d9e9d91-9070-4e08-95e2-83714d549a8d"
-					(reference "R5")
+					(reference "R13")
 					(unit 1)
 				)
@@
 		(dnp no)
 		(fields_autoplaced yes)
-		(property "Reference" "#PWR025"
+		(property "Reference" "#PWR034"
 			(at 104.14 133.35 0)
 			(effects
@@
 			(project "PolicyBadge25"
 				(path "/3911717a-8f19-42c2-8f04-ebfae4e12db6/7d9e9d91-9070-4e08-95e2-83714d549a8d"
-					(reference "#PWR025")
+					(reference "#PWR034")
 					(unit 1)
 				)
@@
 		(dnp no)
 		(fields_autoplaced yes)
-		(property "Reference" "C6"
+		(property "Reference" "C4"
 			(at 157.48 73.66 0)
 			(effects
@@
 			(project ""
 				(path "/3911717a-8f19-42c2-8f04-ebfae4e12db6/7d9e9d91-9070-4e08-95e2-83714d549a8d"
-					(reference "C6")
+					(reference "C4")
 					(unit 1)
 				)
@@
 		(dnp no)
 		(fields_autoplaced yes)
-		(property "Reference" "U3"
+		(property "Reference" "U4"
 			(at 151.13 100.33 0)
 			(effects
@@
 			)
 		)
+		(property "FT Rotation Offset" "180"
+			(at 151.13 110.49 0)
+			(effects
+				(font
+					(size 1.27 1.27)
+				)
+				(hide yes)
+			)
+		)
 		(pin "4"
 		)
@@
 			(project ""
 				(path "/3911717a-8f19-42c2-8f04-ebfae4e12db6/7d9e9d91-9070-4e08-95e2-83714d549a8d"
-					(reference "U3")
+					(reference "U4")
 					(unit 1)
 				)
@@
 		(dnp no)
 		(fields_autoplaced yes)
-		(property "Reference" "C5"
+		(property "Reference" "C7"
 			(at 199.39 116.8399 90)
 			(effects
@@
 			(project "PolicyBadge25"
 				(path "/3911717a-8f19-42c2-8f04-ebfae4e12db6/7d9e9d91-9070-4e08-95e2-83714d549a8d"
-					(reference "C5")
-					(unit 1)
-				)
+					(reference "C7")
+					(unit 1)
+				)

Commit message: Lots of changes, laying out board for board shape
Updated switches
Added headers for XAIO
Fixed Batt Connector polarity
10K pullup on int
Batt monitor resistor divider
Fix buzzer trace
XAIO footprint spacing
Parts:
- renumbered C7 to C10, C3 to C6, C4 to C7, C5 to C8, C6 to C9, L1 to L2, U4 to U6
Changed lines of the file:
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@@
 		(dnp no)
 		(fields_autoplaced yes)
-		(property "Reference" "C6"
+		(property "Reference" "C9"
 			(at 186.69 116.8399 90)
 			(effects
@@
 			(project "PolicyBadge25"
 				(path "/3911717a-8f19-42c2-8f04-ebfae4e12db6/7d9e9d91-9070-4e08-95e2-83714d549a8d"
-					(reference "C6")
+					(reference "C9")
 					(unit 1)
 				)
@@
 		(dnp no)
 		(fields_autoplaced yes)
-		(property "Reference" "#PWR033"
+		(property "Reference" "#PWR038"
 			(at 93.98 133.35 0)
 			(effects
@@
 			(project "PolicyBadge25"
 				(path "/3911717a-8f19-42c2-8f04-ebfae4e12db6/7d9e9d91-9070-4e08-95e2-83714d549a8d"
-					(reference "#PWR033")
+					(reference "#PWR038")
 					(unit 1)
 				)
@@
 		(dnp no)
 		(fields_autoplaced yes)
-		(property "Reference" "#PWR036"
+		(property "Reference" "#PWR041"
 			(at 182.88 133.35 0)
 			(effects
@@
 			(project ""
 				(path "/3911717a-8f19-42c2-8f04-ebfae4e12db6/7d9e9d91-9070-4e08-95e2-83714d549a8d"
-					(reference "#PWR036")
+					(reference "#PWR041")
 					(unit 1)
 				)
@@
 		(dnp no)
 		(fields_autoplaced yes)
-		(property "Reference" "L1"
+		(property "Reference" "L2"
 			(at 115.57 101.6 0)
 			(effects
@@
 			(project ""
 				(path "/3911717a-8f19-42c2-8f04-ebfae4e12db6/7d9e9d91-9070-4e08-95e2-83714d549a8d"
-					(reference "L1")
+					(reference "L2")
 					(unit 1)
 				)
@@
 		(dnp no)
 		(fields_autoplaced yes)
-		(property "Reference" "#PWR035"
+		(property "Reference" "#PWR040"
 			(at 128.27 133.35 0)
 			(effects
@@
 			(project "PolicyBadge25"
 				(path "/3911717a-8f19-42c2-8f04-ebfae4e12db6/7d9e9d91-9070-4e08-95e2-83714d549a8d"
-					(reference "#PWR035")
+					(reference "#PWR040")
 					(unit 1)
 				)
@@
 		(dnp no)
 		(fields_autoplaced yes)
-		(property "Reference" "C5"
+		(property "Reference" "C8"
 			(at 172.72 116.8399 90)
 			(effects
@@
 			(project ""
 				(path "/3911717a-8f19-42c2-8f04-ebfae4e12db6/7d9e9d91-9070-4e08-95e2-83714d549a8d"
-					(reference "C5")
+					(reference "C8")
 					(unit 1)
 				)
@@
 		(dnp no)
 		(fields_autoplaced yes)
-		(property "Reference" "C3"
+		(property "Reference" "C6"
 			(at 107.95 114.2999 90)
 			(effects
@@
 			(project ""
 				(path "/3911717a-8f19-42c2-8f04-ebfae4e12db6/7d9e9d91-9070-4e08-95e2-83714d549a8d"
-					(reference "C3")
+					(reference "C6")
 					(unit 1)
 				)
@@
 		(dnp no)
 		(fields_autoplaced yes)
-		(property "Reference" "#PWR034"
+		(property "Reference" "#PWR039"
 			(at 104.14 133.35 0)
 			(effects
@@
 			(project "PolicyBadge25"
 				(path "/3911717a-8f19-42c2-8f04-ebfae4e12db6/7d9e9d91-9070-4e08-95e2-83714d549a8d"
-					(reference "#PWR034")
+					(reference "#PWR039")
 					(unit 1)
 				)
@@
 		(dnp no)
 		(fields_autoplaced yes)
-		(property "Reference" "C4"
+		(property "Reference" "C7"
 			(at 157.48 73.66 0)
 			(effects
@@
 			(project ""
 				(path "/3911717a-8f19-42c2-8f04-ebfae4e12db6/7d9e9d91-9070-4e08-95e2-83714d549a8d"
-					(reference "C4")
+					(reference "C7")
 					(unit 1)
 				)
@@
 		(dnp no)
 		(fields_autoplaced yes)
-		(property "Reference" "U4"
+		(property "Reference" "U6"
 			(at 151.13 100.33 0)
 			(effects
@@
 			(project ""
 				(path "/3911717a-8f19-42c2-8f04-ebfae4e12db6/7d9e9d91-9070-4e08-95e2-83714d549a8d"
-					(reference "U4")
+					(reference "U6")
 					(unit 1)
 				)
@@
 		(dnp no)
 		(fields_autoplaced yes)
-		(property "Reference" "C7"
+		(property "Reference" "C10"
 			(at 199.39 116.8399 90)
 			(effects
@@
 			(project "PolicyBadge25"
 				(path "/3911717a-8f19-42c2-8f04-ebfae4e12db6/7d9e9d91-9070-4e08-95e2-83714d549a8d"
-					(reference "C7")
-					(unit 1)
-				)
+					(reference "C10")
+					(unit 1)
+				)
